File: product/kicad/clockv7/psu.kicad_sch (KiCad schematic)
At the start: 36 parts, among them CN1 KH-VH-4P-W, J3 Conn_01x02, J4 Conn_01x03, J7 3.5mm, P1 Header-Female-2.54_1x2, Q2 MMBT2222A, U1 SY8388ARHC, U5 CH224K

Commit message: docs(psu): bulletproof v4.1 — worst-case analysis, fix TVS D6, align BOM↔KiCad
- Add worst-case VOUT analysis: ±2.8% (4.86–5.14V) with 1% FB resistors
- Add SY8388ARHC protection specs (UVLO, OVP, OCP, OTP thresholds)
- Add thermal analysis, ripple calculation, capacitor derating analysis
- Fix D6 TVS value in KiCad: SMBJ5.0A → SMBJ24CA (24V, LCSC C19077558)
- Fix TVS package: SMA → SMB (DO-214AA) matching KiCad footprint
- Fix caps LCSC: C52306 (1210) → C12891 (1206) matching KiCad reality
- Fix switching frequency: 500kHz → 600kHz per SY8388A datasheet
- Add KiCad↔docs discrepancy table for reference designators
- Update BOM_VERIFIED.md PSU section to align with all corrections

https://claude.ai/code/session_01MMfczentGLp3AjPWcUBdjF
Parts:
- D6: value SMBJ5.0A -> SMBJ24CA
Changed lines of the file:
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@@
 			)
 		)
-		(property "Value" "SMBJ5.0A"
+		(property "Value" "SMBJ24CA"
 			(at 182.88 67.3099 90)
 			(effects
